File: hardware/ee-02-sensorboard/tk2.sch (EAGLE design)
At the start: 34 parts, among them J1 Debug, J2 AFE3_IDC_CABLE, J3 OPC_N3_CONNECTOR, U11 LM1117-5, U3 EE02, U4 ADS124S08, U5 CHIPCAP2SMD, U6 MAX14830, U7 ORIGIN GPS, U8 EE-NBIOT-01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

Commit message: Updated schematics and layout. Fixed missing common signal on ADC.
Connections:
- net GND: now also U4.AINCOM, U8.GND@2, U8.GND@5
Changed lines of the file:
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@@
 <part name="U$3" library="EE" deviceset="PHOENIX_CONTACT_MSTBVA_2_5" device=""/>
 <part name="GND22" library="supply1" library_urn="urn:adsk.eagle:library:371" deviceset="GND" device=""/>
+<part name="GND23" library="supply1" library_urn="urn:adsk.eagle:library:371" deviceset="GND" device=""/>
 </parts>
 <sheets>
@@
 <instance part="GND21" gate="1" x="203.2" y="2.54"/>
 <instance part="GND22" gate="1" x="276.86" y="38.1"/>
+<instance part="GND23" gate="1" x="210.82" y="55.88"/>
 </instances>
 <busses>
@@
 <pinref part="GND10" gate="1" pin="GND"/>
 <wire x1="119.38" y1="-30.48" x2="119.38" y2="-33.02" width="0.1524" layer="91"/>
+<pinref part="U8" gate="G$1" pin="GND@5"/>
+<wire x1="121.92" y1="-30.48" x2="119.38" y2="-30.48" width="0.1524" layer="91"/>
+<junction x="119.38" y="-30.48"/>
+<pinref part="U8" gate="G$1" pin="GND@2"/>
+<wire x1="124.46" y1="-30.48" x2="121.92" y2="-30.48" width="0.1524" layer="91"/>
+<junction x="121.92" y="-30.48"/>
 </segment>
 <segment>
@@
 <wire x1="271.78" y1="43.18" x2="276.86" y2="43.18" width="0.1524" layer="91"/>
 <wire x1="276.86" y1="43.18" x2="276.86" y2="40.64" width="0.1524" layer="91"/>
+</segment>
+<segment>
+<pinref part="U4" gate="G$1" pin="AINCOM"/>
+<pinref part="GND23" gate="1" pin="GND"/>
+<wire x1="220.98" y1="58.42" x2="210.82" y2="58.42" width="0.1524" layer="91"/>
 </segment>
 </net>
@@
 </sheet>
 </sheets>
+<errors>
+</errors>
 </schematic>
 </drawing>
